File: Circuitry/microcontroller.sch (EAGLE design)
At the start: 0 parts

Commit message: add connections between components
Parts:
- added BOOSTCONVERTER, LED, SWITCH: (no value), pinhead:PINHD-1X2
- added ESP1-15, ESP16-30: (no value), pinhead:PINHD-1X15
- added R1: (no value), rcl:R-US_0207/7
- added SPACER: (no value), pinhead:PINHD-1X10
- added TRANSISTOR: (no value), pinhead:PINHD-1X3
Connections:
- new net N$1: BOOSTCONVERTER.1, ESP1-15.14, LED.1, SWITCH.1
- new net N$2: BOOSTCONVERTER.2, ESP1-15.15, TRANSISTOR.3
- new net N$3: R1.1, TRANSISTOR.2
- new net N$4: ESP16-30.14, R1.2
- new net N$5: ESP16-30.13, SWITCH.2
- new net N$6: LED.2, TRANSISTOR.1
